File: gamepad/gamepad.kicad_pcb (KiCad board)
At the start: 2 copper layers, 100 x 62 mm, 38 parts, among them J1 Conn_01x02_Socket, SW1 SW_SPDT, SW2 SW_Push, SW3 SW_Push, SW4 SW_Push, SW5 SW_Push, SW6 SW_Push, SW7 SW_Push, U1 NE555P, U2 I2C_OLED_MODULE

Commit message: gerber file generated, project is done
Parts:
- added G***: LOGO, LOGO, F.Cu at (164.4, 107.6)
- moved R2 7.45 mm to (84.3, 92.3), turned to 180 degrees
Routing:
- net /BTN_LEFT: track 0.00 -> 120.9 mm
- net /BTN_UP: track 0.00 -> 107.9 mm, vias 0 -> 1
- net +BATT: track 0.00 -> 107.7 mm, vias 0 -> 1
- net +5V: track 0.00 -> 100.7 mm, vias 0 -> 2
- net /BTN_A: track 0.00 -> 80.7 mm
- net /BTN_B: track 0.00 -> 70.8 mm, vias 0 -> 1
- net Net-(C6-Pad1): track 0.00 -> 59.0 mm, vias 0 -> 2
- net Net-(D4-A): track 0.00 -> 56.5 mm, vias 0 -> 1
- net Net-(C7-Pad1): track 0.00 -> 41.9 mm
- net Net-(A1-A5): track 0.00 -> 38.2 mm, vias 0 -> 1
- net Net-(A1-D9): track 0.00 -> 37.3 mm
- net Net-(A1-A4): track 0.00 -> 34.6 mm, vias 0 -> 1
- net Net-(U1-THR): track 0.00 -> 27.7 mm
- net Net-(A1-D4): track 0.00 -> 25.9 mm
- net Net-(A1-D5): track 0.00 -> 20.8 mm
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- added copper zone on B.Cu, net GND
- added copper zone on F.Cu, net GND
Other:
- board text added: "GAMEPAD"
